Commit message: [back] backup before use 231229

File: mdoger7.urdf (robot description, URDF)
Before this commit: robot mdoger7, 13 links, 12 joints
Links:
- added link lb_foot, mass 0.03108367; collision mesh filename=package://mdoger7/meshes/lb_foot.STL; visual mesh filename=package://mdoger7/meshes/lb_foot.STL
- added link lf_foot, mass 0.03108367; collision mesh filename=package://mdoger7/meshes/lf_foot.STL; visual mesh filename=package://mdoger7/meshes/lf_foot.STL
- added link rb_foot, mass 0.03108367; collision mesh filename=package://mdoger7/meshes/rb_foot.STL; visual mesh filename=package://mdoger7/meshes/rb_foot.STL
- added link rf_foot, mass 0.03108367; collision mesh filename=package://mdoger7/meshes/rf_foot.STL; visual mesh filename=package://mdoger7/meshes/rf_foot.STL
- link base_link: mass 3.08231799893906 -> 3.08231817
- link lb1: mass 0.278302034656966 -> 0.27830200
- link lb2: mass 0.444331812401217 -> 0.44448058
- link lb3: mass 0.0675377264543488 -> 0.03645433
- link lf1: mass 0.278302034656967 -> 0.27830200
- link lf2: mass 0.444479146815381 -> 0.44448058
- link lf3: mass 0.0675377262682892 -> 0.03645433
- link rb1: mass 0.278302034656966 -> 0.27830200
- link rb2: mass 0.444100714371199 -> 0.44447934
- link rb3: mass 0.0675377263163792 -> 0.03645433
- link rf1: mass 0.278302034656966 -> 0.27830200
- link rf2: mass 0.444477705439595 -> 0.44447934
- link rf3: mass 0.0675377265651493 -> 0.03645433
Joints:
- added joint lb_foot_joint: type fixed, parent lb3, child lb_foot, origin xyz=-0.14496 -0.14496 0.0001673 rpy=1.5716 0.0008161 2.3562, axis 0 0 0
- added joint lf_foot_joint: type fixed, parent lf3, child lf_foot, origin xyz=-0.14426 -0.14581 0.00072578 rpy=1.5716 0.0008161 2.3562, axis 0 0 0
- added joint rb_foot_joint: type fixed, parent rb3, child rb_foot, origin xyz=0.14496 -0.14496 -0.0001673 rpy=-1.57 -0.0008161 0.7854, axis 0 0 0
- added joint rf_foot_joint: type fixed, parent rf3, child rf_foot, origin xyz=0.14496 -0.14496 -0.0001673 rpy=-1.57 -0.0008161 0.7854, axis 0 0 0
- joint lb1_joint: limit lower=-3.14 upper=3.14 effort=100 velocity=100 -> lower=-0.174 upper=0.174 effort=100 velocity=1; type continuous -> revolute
- joint lb2_joint: axis 0 0 1 -> 0 -0.0011541 -1; limit lower=-3.14 upper=3.14 effort=100 velocity=100 -> lower=-0.523 upper=0.523 effort=100 velocity=1; origin xyz=0.0031 0 -0.069 rpy=3.1404 1.5708 0 -> xyz=0.0031 0.00000358 -0.069 rpy=0 1.5708 0; type continuous -> revolute
- joint lb3_joint: axis 0 0 -1 -> 0 0.0011541 1; limit lower=-3.14 upper=3.14 effort=100 velocity=100 -> lower=-0.523 upper=0.523 effort=100 velocity=1; origin xyz=0.14849 0.14849 -0.0993 rpy=3.1416 0 -3.1416 -> xyz=0.14849 -0.14838 0.099471 rpy=0 0 0; type continuous -> revolute
- joint lf1_joint: axis 0 0 1 -> 0 0 -1; limit lower=-3.14 upper=3.14 effort=100 velocity=100 -> lower=-0.174 upper=0.174 effort=100 velocity=1; origin xyz=0.2043 0.08 0.05825 rpy=-1.5708 0.0011541 1.5708 -> xyz=0.2043 0.08 0.05825 rpy=1.5708 0.0011541 1.5708; type continuous -> revolute
- joint lf2_joint: axis 0 0 1 -> 0 -0.0011541 -1; limit lower=-3.14 upper=3.14 effort=100 velocity=100 -> lower=-0.523 upper=0.523 effort=100 velocity=1; origin xyz=0.0031 0 -0.069 rpy=3.1404 1.5708 0 -> xyz=0.0031 0.00000358 0.069 rpy=0 1.5708 0; type continuous -> revolute
- joint lf3_joint: axis 0 0 -1 -> 0 0.0011541 1; limit lower=-3.14 upper=3.14 effort=100 velocity=100 -> lower=-0.523 upper=0.523 effort=100 velocity=1; origin xyz=-0.14849 -0.14849 -0.0993 rpy=3.1416 0 0 -> xyz=0.14849 -0.14838 0.099471 rpy=0 0 0; type continuous -> revolute
- joint rb1_joint: axis 0 0 1 -> 0 0 -1; limit lower=-3.14 upper=3.14 effort=100 velocity=100 -> lower=-0.174 upper=0.174 effort=100 velocity=1; origin xyz=-0.2043 -0.08 0.05825 rpy=1.5708 0 1.5708 -> xyz=-0.2043 -0.08 0.05825 rpy=1.5708 -0.0011541 -1.5708; type continuous -> revolute
- joint rb2_joint: axis 0 0 1 -> 0 0.0011541 -1; limit lower=-3.14 upper=3.14 effort=100 velocity=100 -> lower=-0.523 upper=0.523 effort=100 velocity=1; origin xyz=-0.0031 0 -0.069 rpy=0 1.5708 0 -> xyz=0.0031 -0.00000358 0.069 rpy=0 1.5708 0; type continuous -> revolute
- joint rb3_joint: axis 0 0.0011541 -1 -> 0 -0.0011541 1; limit lower=-3.14 upper=3.14 effort=0 velocity=0 -> lower=-0.523 upper=0.523 effort=100 velocity=1; origin xyz=0.14849 -0.14849 -0.0993 rpy=3.1404 0 3.1416 -> xyz=-0.14849 -0.14861 0.099129 rpy=0 0 0; type continuous -> revolute
- joint rf1_joint: limit lower=-3.14 upper=3.14 effort=100 velocity=100 -> lower=-0.174 upper=0.174 effort=100 velocity=1; origin xyz=0.2043 -0.08 0.05825 rpy=-1.5708 0.0011541 1.5708 -> xyz=0.2043 -0.08 0.05825 rpy=1.5708 -0.0011541 -1.5708; type continuous -> revolute
- joint rf2_joint: axis 0 0 1 -> 0 0.0011541 -1; limit lower=-3.14 upper=3.14 effort=100 velocity=100 -> lower=-0.523 upper=0.523 effort=100 velocity=1; origin xyz=-0.0031 0 -0.069 rpy=0.0011541 1.5708 0 -> xyz=0.0031 -0.00000358 -0.069 rpy=0 1.5708 0; type continuous -> revolute
- joint rf3_joint: axis 0 0.0011541 -1 -> 0 -0.0011541 1; limit lower=-3.14 upper=3.14 effort=100 velocity=100 -> lower=-0.523 upper=0.523 effort=100 velocity=1; origin xyz=-0.14849 0.14849 -0.0993 rpy=3.1404 0 0 -> xyz=-0.14849 -0.14861 0.099129 rpy=0 0 0; type continuous -> revolute
